File: DesignFiles/WiringDiagrams/EchoCAL-RouterChargeCable/EchoCAL-RouterChargeCable.kicad_sch (KiCad schematic)
At the start: 3 parts

Commit message: documentation update
Connections:
- net NC is gone; now on net GND: J?.2 (Pin_2)
- net +12 VDC: now also J?.1 (Pin_1); no longer J?.5 (Pin_5)
- net GND: no longer J?.1 (Pin_1)
- new net blue: J?.5 (Pin_5)
Other:
- note added: "Bulgin pins SA3348/1"
Changed lines of the file:
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@@
   (title_block
     (title "EchoCAL Router Charge & Comm. Cable")
-    (date "2022-12-08")
+    (date "2023-01-27")
   )
   (no_connect (at 63.5 63.5))
@@
   (no_connect (at 63.5 81.28))
   (no_connect (at 63.5 78.74))
-  (no_connect (at 82.55 66.04))
+  (no_connect (at 123.19 73.66))
   (no_connect (at 63.5 71.12))
   (no_connect (at 63.5 76.2))
@@
     (stroke (width 0) (type default) (color 0 0 0 0))
   )
-  (wire (pts (xy 152.4 63.5) (xy 127 63.5))
+  (wire (pts (xy 152.4 63.5) (xy 104.14 63.5))
+    (stroke (width 0) (type default) (color 0 0 0 0))
+  )
+  (wire (pts (xy 123.19 73.66) (xy 152.4 73.66))
     (stroke (width 0) (type default) (color 0 0 0 0))
   )
@@
     (stroke (width 0) (type default) (color 0 0 0 0))
   )
-  (wire (pts (xy 82.55 66.04) (xy 152.4 66.04))
+  (wire (pts (xy 104.14 63.5) (xy 104.14 101.6))
     (stroke (width 0) (type default) (color 0 0 0 0))
   )
@@
     (stroke (width 0) (type default) (color 0 0 0 0))
   )
-  (wire (pts (xy 63.5 101.6) (xy 129.54 101.6))
+  (wire (pts (xy 63.5 101.6) (xy 104.14 101.6))
     (stroke (width 0) (type default) (color 0 0 0 0))
   )
-  (wire (pts (xy 127 63.5) (xy 127 104.14))
+  (wire (pts (xy 106.68 66.04) (xy 106.68 104.14))
     (stroke (width 0) (type default) (color 0 0 0 0))
   )
-  (wire (pts (xy 152.4 73.66) (xy 129.54 73.66))
+  (wire (pts (xy 106.68 66.04) (xy 152.4 66.04))
     (stroke (width 0) (type default) (color 0 0 0 0))
   )
@@
     (stroke (width 0) (type default) (color 0 0 0 0))
   )
-  (wire (pts (xy 129.54 73.66) (xy 129.54 101.6))
-    (stroke (width 0) (type default) (color 0 0 0 0))
-  )
-  (wire (pts (xy 127 104.14) (xy 63.5 104.14))
+  (wire (pts (xy 63.5 104.14) (xy 106.68 104.14))
     (stroke (width 0) (type default) (color 0 0 0 0))
   )
@@
     (stroke (width 0) (type default) (color 0 0 0 0))
   )
-  (text "Belden 9536 CMG 6C24 shielded cable, 1 m" (at 88.9 59.69 0)
+  (text "Belden 9536 CMG 6C24 shielded cable, 1 m" (at 104.14 59.69 0)
     (effects (font (size 1.27 1.27)) (justify left bottom))
   )
@@
     (effects (font (size 1.27 1.27)) (justify left bottom))
   )
-  (label "red" (at 130.81 73.66 0)
+  (text "Bulgin pins SA3348/1" (at 147.32 82.55 0)
+    (effects (font (size 1.27 1.27)) (justify left bottom))
+  )
+  (label "red" (at 130.81 63.5 0)
     (effects (font (size 1.27 1.27)) (justify left bottom))
   )
@@
     (effects (font (size 1.27 1.27)) (justify left bottom))
   )
-  (label "GND" (at 146.05 63.5 0)
-    (effects (font (size 1.27 1.27)) (justify left bottom))
+  (label "GND{slash}shield" (at 152.4 66.04 180)
+    (effects (font (size 1.27 1.27)) (justify right bottom))
   )
   (label "GND" (at 64.77 104.14 0)
     (effects (font (size 1.27 1.27)) (justify left bottom))
   )
-  (label "blue" (at 130.81 66.04 0)
+  (label "GND" (at 152.4 76.2 180)
+    (effects (font (size 1.27 1.27)) (justify right bottom))
+  )
+  (label "blue" (at 130.81 73.66 0)
     (effects (font (size 1.27 1.27)) (justify left bottom))
   )
@@
     (effects (font (size 1.27 1.27)) (justify left bottom))
   )
+  (label "+V" (at 152.4 63.5 180)
+    (effects (font (size 1.27 1.27)) (justify right bottom))
+  )
   (label "+12 VDC" (at 63.5 101.6 0)
     (effects (font (size 1.27 1.27)) (justify left bottom))
@@
     (effects (font (size 1.27 1.27)) (justify left bottom))
   )
-  (label "black" (at 130.81 63.5 0)
+  (label "black" (at 130.81 66.04 0)
     (effects (font (size 1.27 1.27)) (justify left bottom))
   )
@@
     (effects (font (size 1.27 1.27)) (justify left bottom))
   )
-  (label "NC" (at 146.05 66.04 0)
-    (effects (font (size 1.27 1.27)) (justify left bottom))
-  )
   (symbol (lib_id "Connector:Conn_01x06_Male") (at 157.48 68.58 0) (mirror y) (unit 1)
     (in_bom yes) (on_board yes)
@@
       (effects (font (size 1.27 1.27)) (justify right))
     )
-    (property "Value" "Bulgin PX0410/06P/4550" (id 1) (at 153.67 81.28 0)
+    (property "Value" "Bulgin PX0410/06P/4550" (id 1) (at 147.32 78.74 0)
       (effects (font (size 1.27 1.27)) (justify right))
     )
